Commit message: modify MJCF, URDF

File: rby1a/urdf/model.urdf (robot description, URDF)
Before this commit: robot RB_Y1_V1.0.1, 34 links, 33 joints
Links:
- removed link link_torso_5
- added link link_torso_base, mass 2.24282123; collision capsule coltype=1 length=0.230 radius=0.105; visual mesh filename=./meshes/LINK_1.dae
- link link_torso_0: mass 2.24282123 -> 9.72162676; geometry collision capsule coltype=2 length=0.220 radius=0.115; visual mesh filename=./meshes/LINK_2.dae
- link link_torso_1: mass 9.72162676 -> 9.21691850; geometry collision capsule coltype=4 length=0.1600 radius=0.095; visual mesh filename=./meshes/LINK_3.dae
- link link_torso_2: mass 9.21691850 -> 4.18679196; geometry visual mesh filename=./meshes/LINK_4.dae
- link link_torso_3: mass 4.18679196 -> 4.45566276; geometry collision capsule coltype=8 length=0.2 radius=0.105; visual mesh filename=./meshes/LINK_5.dae
- link link_torso_4: mass 4.45566276 -> 12.59012341; geometry collision capsule coltype=16 length=0.1350 radius=0.155; visual mesh filename=./meshes/LINK_6.dae
Joints:
- removed joint torso_5
- added joint torso_base: type fixed, parent base, child link_torso_base, origin xyz=0.0 0.0 0.2805 rpy=0.0 0.0 0.0, axis 1 0 0
- joint head_base: parent link_torso_5 -> link_torso_4
- joint left_arm_0: parent link_torso_5 -> link_torso_4
- joint right_arm_0: parent link_torso_5 -> link_torso_4
- joint torso_0: axis 1 0 0 -> 0 1 0; limit lower=-0.261799388 upper=0.261799388 effort=270.0 velocity=2.09439510 -> lower=-0.523598776 upper=1.570796327 effort=270.0 velocity=2.09439510; origin xyz=0.0 0.0 0.2805 rpy=0.0 0.0 0.0 -> xyz=0.0 0.0 0.0 rpy=0.0 0.0 0.0; parent base -> link_torso_base
- joint torso_1: limit lower=-0.523598776 upper=1.570796327 effort=270.0 velocity=2.09439510 -> lower=-2.617993878 upper=1.570796327 effort=270.0 velocity=2.09439510; origin xyz=0.0 0.0 0.0 rpy=0.0 0.0 0.0 -> xyz=0.0 0.0 0.350 rpy=0.0 0.0 0.0
- joint torso_2: limit lower=-2.617993878 upper=1.570796327 effort=270.0 velocity=2.09439510 -> lower=-0.785398163 upper=1.570796327 effort=120.0 velocity=3.141592654
- joint torso_3: axis 0 1 0 -> 1 0 0; limit lower=-0.785398163 upper=1.570796327 effort=120.0 velocity=3.141592654 -> lower=-0.523598776 upper=0.523598776 effort=120.0 velocity=3.141592654; origin xyz=0.0 0.0 0.350 rpy=0.0 0.0 0.0 -> xyz=0.0 0.0 0.0 rpy=0.0 0.0 0.0
- joint torso_4: axis 1 0 0 -> 0 0 1; limit lower=-0.523598776 upper=0.523598776 effort=120.0 velocity=3.141592654 -> lower=-2.35619449 upper=2.35619449 effort=120.0 velocity=3.141592654; origin xyz=0.0 0.0 0.0 rpy=0.0 0.0 0.0 -> xyz=0.0 0.0 0.309426548461 rpy=0.0 0.0 0.0
